File: Allwinner_V3S_Spotify/Allwinner_V3S_Spotify.kicad_sch (KiCad schematic)
At the start: 0 parts

Commit message: More work on Schematics
Other:
- added sheet Connectivity (Connectivity.kicad_sch)
- added sheet Power (Power.kicad_sch)
Changed lines of the file:
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@@
 	(paper "A4")
+	(sheet
+		(at 221.996 98.806)
+		(size 43.942 44.45)
+		(fields_autoplaced yes)
+		(stroke
+			(width 0.1524)
+			(type solid)
+		)
+		(fill
+			(color 0 0 0 0.0000)
+		)
+		(property "Sheetname" "Power"
+			(at 221.996 98.0944 0)
+			(effects
+				(font
+					(size 1.27 1.27)
+				)
+				(justify left bottom)
+			)
+		)
+		(property "Sheetfile" "Power.kicad_sch"
+			(at 221.996 143.8406 0)
+			(effects
+				(font
+					(size 1.27 1.27)
+				)
+				(justify left top)
+			)
+		)
+		(instances
+			(project "Allwinner_V3S_Spotify"
+				(path "/149e8d94-e7c7-4bd7-93a7-37c7815b68ab"
+					(page "4")
+				)
+			)
+		)
+	)
 	(sheet
 		(at 43.942 106.172)
@@
 				)
 			)
+		)
+	)
+	(sheet
+		(at 32.258 25.908)
+		(size 65.024 47.244)
+		(fields_autoplaced yes)
+		(stroke
+			(width 0.1524)
+			(type solid)
+		)
+		(fill
+			(color 0 0 0 0.0000)
+		)
+		(property "Sheetname" "Connectivity"
+			(at 32.258 25.1964 0)
+			(effects
+				(font
+					(size 1.27 1.27)
+				)
+				(justify left bottom)
+			)
+		)
+		(property "Sheetfile" "Connectivity.kicad_sch"
+			(at 32.258 73.7366 0)
+			(effects
+				(font
+					(size 1.27 1.27)
+				)
+				(justify left top)
+			)
+		)
+		(instances
+			(project "Allwinner_V3S_Spotify"
+				(path "/149e8d94-e7c7-4bd7-93a7-37c7815b68ab"
+					(page "5")
+				)
+			)
