File: Allwinner_V3S_Spotify/LCD.kicad_sch (KiCad schematic)
At the start: 1 part, among them J1 54104-4031

Commit message: More work on Schematics
Connections:
- net GND: now reaches J1.1
- net GND: now also J1.29, J1.3, J1.36
- net LCD_R5: now reaches J1.10
- net LCD_R6: now reaches J1.11
- net LCD_R7: now reaches J1.12
- net LCD_G0: now reaches J1.13
- net LCD_G1: now reaches J1.14
- net LCD_G2: now reaches J1.15
- net LCD_G3: now reaches J1.16
- net LCD_G4: now reaches J1.17
- net LCD_G5: now reaches J1.18
- net LCD_G6: now reaches J1.19
- net VLCD: now reaches J1.2
- net LCD_G7: now reaches J1.20
- net LCD_B0: now reaches J1.21
- net LCD_B1: now reaches J1.22
- net LCD_B2: now reaches J1.23
- net LCD_B3: now reaches J1.24
- net LCD_B4: now reaches J1.25
- net LCD_B5: now reaches J1.26
- net LCD_B6: now reaches J1.27
- net LCD_B7: now reaches J1.28
- net LCD_CLK: now reaches J1.30
- net LCD_DISP: now reaches J1.31
- net LCD_HSYNC: now reaches J1.32
- net LCD_VSYNC: now reaches J1.33
- net LCD_DEN: now reaches J1.34
- net LCD_BIST: now reaches J1.35
- net LCD_NC: now reaches J1.37
- net LCD_NC: now also J1.38, J1.39, J1.40
- net +3.3V: now reaches J1.4
- net LCD_R0: now reaches J1.5
- net LCD_R1: now reaches J1.6
- net LCD_R2: now reaches J1.7
- net LCD_R3: now reaches J1.8
- net LCD_R4: now reaches J1.9
