File: Allwinner_V3S_Spotify/Connectivity.kicad_sch (KiCad schematic)
At the start: 15 parts, among them J2 USB_A, J3 Micro_SD_Card_Det2

Commit message: More Schematics
Parts:
- added C15, C16: 100nF, Capacitor_SMD:C_0603_1608Metric_Pad1.08x0.95mm_HandSolder, symbol Device:C_Small
- added J5: RJ45_Wuerth_7499010121A, Connector_RJ:RJ45_Wuerth_7499010121A_Horizontal, symbol Connector:RJ45_Wuerth_7499010121A
- added R21: 0R, Resistor_SMD:R_01005_0402Metric, symbol Device:R_Small
- added R22, R23, R28, R29: 50R, Resistor_SMD:R_01005_0402Metric, symbol Device:R_Small
- added R24, R25: 270R, Resistor_SMD:R_01005_0402Metric, symbol Device:R_Small
Connections:
- net +3V3: now also R21.1
- net GND: now also J2.4 (GND), J2.5 (Shield), C15.2, C16.1, J5.11, J5.8, J5.9, J5.SH
- net VBUS: now reaches J2.1 (VBUS)
- net USB_D-: now reaches J2.2 (D-)
- net USB_D+: now reaches J2.3 (D+)
- new net: J5.10, R25.2
- new net: J5.12, R24.2
- new net: J5.2 (TCT), J5.5 (RCT), R21.2
- new net: C16.2, R28.2, R29.1
- new net: C15.1, R22.1, R23.2
- new net ETH_GRN_LED: R25.1
- new net ETH_RD+: J5.4 (RD+), R28.1
- new net ETH_RD-: J5.6 (RD-), R29.2
- new net ETH_TD+: J5.1 (TD+), R23.1
- new net ETH_TD-: J5.3 (TD-), R22.2
- new net ETH_YEL_LED: R24.1
Other:
- moved on the sheet: J2
