File: Allwinner_V3S_Spotify/Power.kicad_sch (KiCad schematic)
At the start: 8 parts, among them U2 EA3058, U3 AP3012

Commit message: More Schematics
Parts:
- removed U2: EA3058, Package_DFN_QFN:QFN-24-1EP_4x4mm_P0.5mm_EP2.65x2.65mm, symbol Allwinner_V3S_Spotify:EA3058
- added C10, C4, C6, C8: 10uF, symbol Device:C_Small
- added C11, C12, C13, C14: 22uF, symbol Device:C_Small
- added C3, C5, C7, C9: 100nF, Capacitor_SMD:C_0603_1608Metric_Pad1.08x0.95mm_HandSolder, symbol Device:C_Small
- added J4: Conn_01x02_Socket, Connector_JST:JST_XH_S2B-XH-A-1_1x02_P2.50mm_Horizontal, symbol Connector:Conn_01x02_Socket
- added L2: 1uH, symbol Device:L
- added L3: 1u5, symbol Device:L
- added L4: 2uH, symbol Device:L
- added L5: 2u2, symbol Device:L
- added R10, R12, R16: 10K, Resistor_SMD:R_0603_1608Metric_Pad0.98x0.95mm_HandSolder, symbol Device:R
- added R11: 12K4, Resistor_SMD:R_0603_1608Metric_Pad0.98x0.95mm_HandSolder, symbol Device:R
- added R13: 33K, Resistor_SMD:R_0603_1608Metric_Pad0.98x0.95mm_HandSolder, symbol Device:R
- added R14: 12K, Resistor_SMD:R_0603_1608Metric_Pad0.98x0.95mm_HandSolder, symbol Device:R
- added R15: 31K6, Resistor_SMD:R_0603_1608Metric_Pad0.98x0.95mm_HandSolder, symbol Device:R
- added R17, R18, R19, R20: 0R, Resistor_SMD:R_0603_1608Metric_Pad0.98x0.95mm_HandSolder, symbol Device:R
- added R9: 4K99, Resistor_SMD:R_0603_1608Metric_Pad0.98x0.95mm_HandSolder, symbol Device:R
- added U2, U4, U5, U6: AP62250WU, Package_TO_SOT_SMD:TSOT-23-6, symbol Regulator_Switching:AP62250WU
Connections:
- net GND: now also C10.2, C11.2, C12.2, C13.2, C14.2, C4.2, C6.2, C8.2, J4.2 (Pin_2), R10.2, R12.2, R14.2, R16.2, U2.1 (GND), U4.1 (GND), U5.1 (GND), U6.1 (GND)
- new net: C3.2, L2.1, U4.2 (SW)
- new net: R10.1, R9.2, U4.4 (FB)
- new net: C3.1, U4.6 (BST)
- new net: C14.1, L5.2, R15.1, R20.1
- new net: C11.1, L2.2, R17.1, R9.1
- new net: C9.2, L5.1, U6.2 (SW)
- new net: R15.2, R16.1, U6.4 (FB)
- new net: C9.1, U6.6 (BST)
- new net: C12.1, L3.2, R11.1, R18.1
- new net: R11.2, R12.1, U2.4 (FB)
- new net: R13.2, R14.1, U5.4 (FB)
- new net: C13.1, L4.2, R13.1, R19.1
- new net: C7.1, U5.6 (BST)
- new net: C7.2, L4.1, U5.2 (SW)
- new net: C5.2, L3.1, U2.2 (SW)
- new net: C5.1, U2.6 (BST)
- new net +1V2: R17.2
- new net +1V8: R18.2
- new net +3V0: R19.2
- new net +3V3: R20.2
- new net VIN: C10.1, C4.1, C6.1, C8.1, J4.1 (Pin_1), U2.3 (VIN), U4.3 (VIN), U5.3 (VIN), U6.3 (VIN)
Other:
- note added: "EN CAN BE FLOATING"
- note added: "L = (VOUT(VIN - VOUT)) / VIN DELTA_IL Fsw"
- note added: "R1 = R2((VOUT/0.8V)-1)"
